Commit message: urdf_update_tf_setup

File: zenorak_ros2_control/description/zenorak.xacro (robot description, xacro)
@@ -1,14 +1,24 @@
 <?xml version="1.0" encoding="utf-8"?>
-<robot xmlns:xacro="http://ros.org/wiki/xacro" name="zenorak">
+<robot name="zenorak_ros2_control"
+    xmlns:xacro="http://www.ros.org/wiki/xacro">
+    <!-- Start GZ or Ignition depending on ROS 2 Version -->
+    <xacro:arg name="is_ignition" default="true"/>
+    <link name="base_footprint"/>
+    <joint name="base_footprint_part" type="fixed">
+        <origin xyz="-0.4763649 0.3169183 0.179" rpy="0 0 0"/>
+        <parent link="base_footprint"/>
+        <child link="base_link"/>
+    </joint>
+    <!-- ================= BASE LINK ================= -->
     <link name="base_link">
         <inertial>
             <origin xyz="0.225609050013199 -0.382431512154995 0.110457297768854" rpy="0 0 0" />
             <mass value="37.6020822567643" />
-            <inertia ixx="0.918856210506478" ixy="-0.0965949212708132" ixz="0.0494096588148493" iyy="3.15876696877023" iyz="0.0144413623668442" izz="3.60003819027792" />
-        </inertial>
-        <visual>
-            <origin xyz="0 0 0" rpy="0 0 0" />
-            <geometry>
-                <mesh filename="file://$(find zenorak_ros2_control)/meshes/base_link.STL" />
+            <inertia ixx="0.918856210506479" ixy="-0.0965949212708133" ixz="0.0494096588148494" iyy="3.15876696877023" iyz="0.0144413623668441" izz="3.60003819027792" />
+        </inertial>
+        <visual>
+            <origin xyz="0 0 0" rpy="0 0 0" />
+            <geometry>
+                <mesh filename="package://zenorak_ros2_control/meshes/base_link.STL" />
             </geometry>
             <material name="">
@@ -19,18 +29,18 @@
             <origin xyz="0 0 0" rpy="0 0 0" />
             <geometry>
-                <mesh filename="file://$(find zenorak_ros2_control)/meshes/base_link.STL" />
-            </geometry>
-        </collision>
-    </link>
-    <link name="rear_wheel_left">
-        <inertial>
-            <origin xyz="-0.0679260215961158 2.36125695107781E-07 -1.9473195911994E-06" rpy="0 0 0" />
-            <mass value="7.07873349857203" />
-            <inertia ixx="0.080850131713722" ixy="1.35417971922918E-10" ixz="-9.3394289632707E-10" iyy="0.0480312798741648" iyz="5.10051862520795E-08" izz="0.0480308658130902" />
-        </inertial>
-        <visual>
-            <origin xyz="0 0 0" rpy="0 0 0" />
-            <geometry>
-                <mesh filename="file://$(find zenorak_ros2_control)/meshes/rear_wheel_left.STL" />
+                <mesh filename="package://zenorak_ros2_control/meshes/base_link.STL" />
+            </geometry>
+        </collision>
+    </link>
+    <link name="rear_wheel_left_part">
+        <inertial>
+            <origin xyz="-0.0679260215961148 2.36125695066147E-07 -1.94731959117164E-06" rpy="0 0 0" />
+            <mass value="7.07873349857202" />
+            <inertia ixx="0.080850131713722" ixy="1.35417971474635E-10" ixz="-9.33942895770876E-10" iyy="0.0480312798741648" iyz="5.10051862542479E-08" izz="0.0480308658130902" />
+        </inertial>
+        <visual>
+            <origin xyz="0 0 0" rpy="0 0 0" />
+            <geometry>
+                <mesh filename="package://zenorak_ros2_control/meshes/rear_wheel_left_part.STL" />
             </geometry>
             <material name="">
@@ -41,5 +51,5 @@
             <origin xyz="0 0 0" rpy="0 0 0" />
             <geometry>
-                <mesh filename="file://$(find zenorak_ros2_control)/meshes/rear_wheel_left.STL" />
+                <mesh filename="package://zenorak_ros2_control/meshes/rear_wheel_left_part.STL" />
             </geometry>
         </collision>
@@ -48,17 +58,17 @@
         <origin xyz="-0.112759182276568 -0.562875460951289 -0.0350858656525844" rpy="3.0811708109372 0 1.5707963267949" />
         <parent link="base_link" />
-        <child link="rear_wheel_left" />
+        <child link="rear_wheel_left_part" />
         <axis xyz="1 0 0" />
     </joint>
-    <link name="rear_wheel_right">
-        <inertial>
-            <origin xyz="0.0703369302084167 -2.36126483685317E-07 -1.94731702234802E-06" rpy="0 0 0" />
+    <link name="rear_wheel_right_part">
+        <inertial>
+            <origin xyz="0.0703369302084167 -2.36126483657562E-07 -1.94731702234455E-06" rpy="0 0 0" />
             <mass value="7.07873349872348" />
-            <inertia ixx="0.0808501317144986" ixy="-1.35425404064983E-10" ixz="-9.3394364160223E-10" iyy="0.0480312798744027" iyz="-5.10057398585024E-08" izz="0.0480308658136232" />
-        </inertial>
-        <visual>
-            <origin xyz="0 0 0" rpy="0 0 0" />
-            <geometry>
-                <mesh filename="file://$(find zenorak_ros2_control)/meshes/rear_wheel_right.STL" />
+            <inertia ixx="0.0808501317144986" ixy="-1.35425404030724E-10" ixz="-9.33943641692648E-10" iyy="0.0480312798744027" iyz="-5.10057398585024E-08" izz="0.0480308658136232" />
+        </inertial>
+        <visual>
+            <origin xyz="0 0 0" rpy="0 0 0" />
+            <geometry>
+                <mesh filename="package://zenorak_ros2_control/meshes/rear_wheel_right_part.STL" />
             </geometry>
             <material name="">
@@ -69,5 +79,5 @@
             <origin xyz="0 0 0" rpy="0 0 0" />
             <geometry>
-                <mesh filename="file://$(find zenorak_ros2_control)/meshes/rear_wheel_right.STL" />
+                <mesh filename="package://zenorak_ros2_control/meshes/rear_wheel_right_part.STL" />
             </geometry>
         </collision>
@@ -76,17 +86,17 @@
         <origin xyz="-0.112759182276568 -0.0709611226931948 -0.0350858656525845" rpy="-3.0811708109372 0 -1.5707963267949" />
         <parent link="base_link" />
-        <child link="rear_wheel_right" />
-        <axis xyz="1 0 0" />
-    </joint>
-    <link name="front_wheel_left">
-        <inertial>
-            <origin xyz="-0.0679260215959383 -1.30981837784261E-06 1.46020001273728E-06" rpy="0 0 0" />
+        <child link="rear_wheel_right_part" />
+        <axis xyz="-1 0 0" />
+    </joint>
+    <link name="front_wheel_left_part">
+        <inertial>
+            <origin xyz="-0.0679260215959383 -1.30981837787036E-06 1.46020001273728E-06" rpy="0 0 0" />
             <mass value="7.07873349856122" />
-            <inertia ixx="0.0808501317136931" ixy="-6.4636167255867E-10" ixz="6.87611674264496E-10" iyy="0.0480310958801467" iyz="2.11972896282595E-07" izz="0.0480310498070746" />
-        </inertial>
-        <visual>
-            <origin xyz="0 0 0" rpy="0 0 0" />
-            <geometry>
-                <mesh filename="file://$(find zenorak_ros2_control)/meshes/front_wheel_left.STL" />
+            <inertia ixx="0.0808501317136931" ixy="-6.46361672812888E-10" ixz="6.87611674322253E-10" iyy="0.0480310958801467" iyz="2.1197289628086E-07" izz="0.0480310498070746" />
+        </inertial>
+        <visual>
+            <origin xyz="0 0 0" rpy="0 0 0" />
+            <geometry>
+                <mesh filename="package://zenorak_ros2_control/meshes/front_wheel_left_part.STL" />
             </geometry>
             <material name="">
@@ -97,5 +107,5 @@
             <origin xyz="0 0 0" rpy="0 0 0" />
             <geometry>
-                <mesh filename="file://$(find zenorak_ros2_control)/meshes/front_wheel_left.STL" />
+                <mesh filename="package://zenorak_ros2_control/meshes/front_wheel_left_part.STL" />
             </geometry>
         </collision>
@@ -104,17 +114,17 @@
         <origin xyz="0.476364897342864 -0.562875460951289 -0.0350858656525772" rpy="-1.93646547797082 0 1.5707963267949" />
         <parent link="base_link" />
-        <child link="front_wheel_left" />
+        <child link="front_wheel_left_part" />
         <axis xyz="1 0 0" />
     </joint>
-    <link name="front_wheel_right">
-        <inertial>
-            <origin xyz="0.0703369302085942 1.30981749490999E-06 1.4601974790418E-06" rpy="0 0 0" />
+    <link name="front_wheel_right_part">
+        <inertial>
+            <origin xyz="0.0703369302085943 1.30981749479897E-06 1.46019747881976E-06" rpy="0 0 0" />
             <mass value="7.07873349871121" />
-            <inertia ixx="0.0808501317144757" ixy="6.46368421612624E-10" ixz="6.87608507545178E-10" iyy="0.0480310958799598" iyz="-2.11972948763184E-07" izz="0.048031049808038" />
-        </inertial>
-        <visual>
-            <origin xyz="0 0 0" rpy="0 0 0" />
-            <geometry>
-                <mesh filename="file://$(find zenorak_ros2_control)/meshes/front_wheel_right.STL" />
+            <inertia ixx="0.0808501317144757" ixy="6.4636842171885E-10" ixz="6.87608507579504E-10" iyy="0.0480310958799598" iyz="-2.11972948770123E-07" izz="0.048031049808038" />
+        </inertial>
+        <visual>
+            <origin xyz="0 0 0" rpy="0 0 0" />
+            <geometry>
+                <mesh filename="package://zenorak_ros2_control/meshes/front_wheel_right_part.STL" />
             </geometry>
             <material name="">
@@ -125,5 +135,5 @@
             <origin xyz="0 0 0" rpy="0 0 0" />
             <geometry>
-                <mesh filename="file://$(find zenorak_ros2_control)/meshes/front_wheel_right.STL" />
+                <mesh filename="package://zenorak_ros2_control/meshes/front_wheel_right_part.STL" />
             </geometry>
         </collision>
@@ -132,118 +142,128 @@
         <origin xyz="0.476364897342864 -0.0709611226931948 -0.0350858656525772" rpy="1.93646547797082 0 -1.5707963267949" />
         <parent link="base_link" />
-        <child link="front_wheel_right" />
+        <child link="front_wheel_right_part" />
         <axis xyz="1 0 0" />
     </joint>
-    <link name="manipulator_base">
-        <inertial>
-            <origin xyz="0.157263621201152 0.101352922065795 1.87079851476923E-06" rpy="0 0 0" />
-            <mass value="2.2590906062532" />
-            <inertia ixx="0.00386029628578382" ixy="0.000859869774009775" ixz="-3.86394674955334E-08" iyy="0.0106698133064369" iyz="-2.29733762474938E-07" izz="0.00878688353686422" />
-        </inertial>
-        <visual>
-            <origin xyz="0 0 0" rpy="0 0 0" />
-            <geometry>
-                <mesh filename="file://$(find zenorak_ros2_control)/meshes/manipulator_base.STL" />
-            </geometry>
-            <material name="">
-                <color rgba="0.698039215686274 0.698039215686274 0.698039215686274 1" />
-            </material>
-        </visual>
-        <collision>
-            <origin xyz="0 0 0" rpy="0 0 0" />
-            <geometry>
-                <mesh filename="file://$(find zenorak_ros2_control)/meshes/manipulator_base.STL" />
+    <!-- ================= MANIPULATOR ================= -->
+    <!-- (unchanged from your original URDF) -->
+    <xacro:property name="PI" value="3.14159265359" />
+    <xacro:property name="effort" value="30.0" />
+    <xacro:property name="velocity" value="10.0" />
+    <link name="manipulator_base_part">
+        <inertial>
+            <origin xyz="0.157263621201152 0.101352922065795 1.87079851471372E-06" rpy="0 0 0"/>
+            <mass value="2.2590906062532"/>
+            <inertia ixx="0.00386029628578382" ixy="0.000859869774009775" ixz="-3.86394674955561E-08" iyy="0.0106698133064369" iyz="-2.29733762474938E-07" izz="0.00878688353686422"/>
+        </inertial>
+        <visual>
+            <origin xyz="0 0 0" rpy="0 0 0"/>
+            <geometry>
+                <mesh filename="package://zenorak_ros2_control/meshes/manipulator_base_part.STL"/>
+            </geometry>
+            <material name="">
+                <color rgba="0.698039215686274 0.698039215686274 0.698039215686274 1"/>
+            </material>
+        </visual>
+        <collision>
+            <origin xyz="0 0 0" rpy="0 0 0"/>
+            <geometry>
+                <mesh filename="package://zenorak_ros2_control/meshes/manipulator_base_part.STL"/>
             </geometry>
         </collision>
     </link>
     <joint name="manipulator_base" type="fixed">
-        <origin xyz="0.285562617252501 -0.383543373894075 0.122214368843715" rpy="1.5707963267949 0 0" />
-        <parent link="base_link" />
-        <child link="manipulator_base" />
-        <axis xyz="0 0 0" />
-    </joint>
-    <link name="linkk_1">
-        <inertial>
-            <origin xyz="0.0967880571495806 0.260782714032567 5.34932605100735E-06" rpy="0 0 0" />
-            <mass value="0.30570759973379" />
-            <inertia ixx="0.000992147641054961" ixy="-0.000647770727662863" ixz="-2.0905494412407E-08" iyy="0.00145140179568686" iyz="-5.0163866836673E-11" izz="0.00241244142666066" />
-        </inertial>
-        <visual>
-            <origin xyz="0 0 0" rpy="0 0 0" />
-            <geometry>
-                <mesh filename="file://$(find zenorak_ros2_control)/meshes/linkk_1.STL" />
-            </geometry>
-            <material name="">
-                <color rgba="0.792156862745098 0.819607843137255 0.933333333333333 1" />
-            </material>
-        </visual>
-        <collision>
-            <origin xyz="0 0 0" rpy="0 0 0" />
-            <geometry>
-                <mesh filename="file://$(find zenorak_ros2_control)/meshes/linkk_1.STL" />
-            </geometry>
-        </collision>
-    </link>
-    <joint name="linkk_1" type="continuous">
-        <origin xyz="0.201025284688791 0.11855300220073 0" rpy="0 0 -0.285822234578718" />
-        <parent link="manipulator_base" />
-        <child link="linkk_1" />
-        <axis xyz="0 0 1" />
-    </joint>
-    <link name="link_2">
-        <inertial>
-            <origin xyz="0.00878775849458258 -0.0734961309869711 2.07355477732651E-07" rpy="0 0 0" />
-            <mass value="0.175654601701013" />
-            <inertia ixx="0.000573214810454448" ixy="3.03938118267286E-06" ixz="8.82691411511942E-09" iyy="6.94547105212176E-05" iyz="9.92533331171897E-08" izz="0.000603952650743279" />
-        </inertial>
-        <visual>
-            <origin xyz="0 0 0" rpy="0 0 0" />
-            <geometry>
-                <mesh filename="file://$(find zenorak_ros2_control)/meshes/link_2.STL" />
-            </geometry>
-            <material name="">
-                <color rgba="0.792156862745098 0.819607843137255 0.933333333333333 1" />
-            </material>
-        </visual>
-        <collision>
-            <origin xyz="0 0 0" rpy="0 0 0" />
-            <geometry>
-                <mesh filename="file://$(find zenorak_ros2_control)/meshes/link_2.STL" />
-            </geometry>
-        </collision>
-    </link>
-    <joint name="link_2" type="continuous">
-        <origin xyz="0.344393779505362 0.432597470756819 0" rpy="0 0 1.10459913734809" />
-        <parent link="linkk_1" />
-        <child link="link_2" />
-        <axis xyz="0 0 1" />
-    </joint>
-    <link name="link_3">
-        <inertial>
-            <origin xyz="1.89394355049055E-05 -0.0795967370192067 0.0218929431449237" rpy="0 0 0" />
-            <mass value="1.17447274540729" />
-            <inertia ixx="0.00484793799004324" ixy="1.17794795886164E-05" ixz="-2.18730896943588E-06" iyy="0.00375075117691504" iyz="0.00097675661116565" izz="0.00268332926346937" />
-        </inertial>
-        <visual>
-            <origin xyz="0 0 0" rpy="0 0 0" />
-            <geometry>
-                <mesh filename="file://$(find zenorak_ros2_control)/meshes/link_3.STL" />
-            </geometry>
-            <material name="">
-                <color rgba="0.298039215686275 0.298039215686275 0.298039215686275 1" />
-            </material>
-        </visual>
-        <collision>
-            <origin xyz="0 0 0" rpy="0 0 0" />
-            <geometry>
-                <mesh filename="file://$(find zenorak_ros2_control)/meshes/link_3.STL" />
-            </geometry>
-        </collision>
-    </link>
-    <joint name="link_3" type="continuous">
-        <origin xyz="0 -0.291104719303414 0" rpy="2.3649900417239 -1.5707963267949 0" />
-        <parent link="link_2" />
-        <child link="link_3" />
-        <axis xyz="1 0 0" />
+        <origin xyz="0.285562617252501 -0.383543373894075 0.122214368843715" rpy="1.5707963267949 0 0"/>
+        <parent link="base_link"/>
+        <child link="manipulator_base_part"/>
+        <axis xyz="0 0 0"/>
+    </joint>
+    <link name="linkk_1_part">
+        <inertial>
+            <origin xyz="0.0967880608316517 0.260782714993558 5.34841523558427E-06" rpy="0 0 0"/>
+            <mass value="0.305707588406735"/>
+            <inertia ixx="0.000992147501244408" ixy="-0.000647770730773342" ixz="-2.09054739391165E-08" iyy="0.00145140179560872" iyz="-5.06820595760279E-11" izz="0.0024124412867919"/>
+        </inertial>
+        <visual>
+            <origin xyz="0 0 0" rpy="0 0 0"/>
+            <geometry>
+                <mesh filename="package://zenorak_ros2_control/meshes/linkk_1_part.STL"/>
+            </geometry>
+            <material name="">
+                <color rgba="0.792156862745098 0.819607843137255 0.933333333333333 1"/>
+            </material>
+        </visual>
+        <collision>
+            <origin xyz="0 0 0" rpy="0 0 0"/>
+            <geometry>
+                <mesh filename="package://zenorak_ros2_control/meshes/linkk_1_part.STL"/>
+            </geometry>
+        </collision>
+    </link>
+    <joint name="linkk_1" type="revolute">
+        <origin xyz="0.201025284688791 0.11855300220073 0" rpy="0 0 -0.285822234578718"/>
+        <parent link="manipulator_base_part"/>
+        <child link="linkk_1_part"/>
+        <axis xyz="0 0 1"/>
+        <limit lower="${0.001}" upper="-${0.8}" effort="${effort}" velocity="${velocity}"/>
+    </joint>
+    <link name="link_2_part">
+        <inertial>
+            <origin xyz="0.00878775849458302 -0.0734961309869713 2.07355477566118E-07" rpy="0 0 0"/>
+            <mass value="0.175654601701013"/>
+            <inertia ixx="0.000573214810454448" ixy="3.03938118267296E-06" ixz="8.82691411511877E-09" iyy="6.94547105212174E-05" iyz="9.92533331171933E-08" izz="0.000603952650743279"/>
+        </inertial>
+        <visual>
+            <origin xyz="0 0 0" rpy="0 0 0"/>
+            <geometry>
+                <mesh filename="package://zenorak_ros2_control/meshes/link_2_part.STL"/>
+            </geometry>
+            <material name="">
+                <color rgba="0.792156862745098 0.819607843137255 0.933333333333333 1"/>
+            </material>
+        </visual>
+        <collision>
+            <origin xyz="0 0 0" rpy="0 0 0"/>
+            <geometry>
+                <mesh filename="package://zenorak_ros2_control/meshes/link_2_part.STL"/>
+            </geometry>
+        </collision>
+    </link>
+    <!-- CHANGED: continuous -> revolute + limits -->
+    <joint name="link_2" type="revolute">
+        <origin xyz="0.344393779505362 0.432597470756819 0" rpy="0 0 1.10459913734809"/>
+        <parent link="linkk_1_part"/>
+        <child link="link_2_part"/>
+        <axis xyz="0 0 1"/>
+        <limit lower="${0.195}" upper="-${1.129}" effort="${effort}" velocity="${velocity}"/>
+    </joint>
+    <link name="link_3_part">
+        <inertial>
+            <origin xyz="1.89394355052941E-05 -0.0795967370189372 0.0218929431451993" rpy="0 0 0"/>
+            <mass value="1.1744727454073"/>
+            <inertia ixx="0.00484793799004943" ixy="1.17794795886547E-05" ixz="-2.18730896944459E-06" iyy="0.00375075117692043" iyz="0.000976756611162925" izz="0.00268332926347022"/>
+        </inertial>
+        <visual>
+            <origin xyz="0 0 0" rpy="0 0 0"/>
+            <geometry>
+                <mesh filename="package://zenorak_ros2_control/meshes/link_3_part.STL"/>
+            </geometry>
+            <material name="">
+                <color rgba="0.298039215686275 0.298039215686275 0.298039215686275 1"/>
+            </material>
+        </visual>
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